Commit message: update URDF frame, SRDF home pose, launch files, and add JAKA action server

File: urdf/dual_arm.urdf.xacro (robot description, xacro)
@@ -7,5 +7,5 @@
     <parent link="world"/>
     <child link="left_base_link"/>
-    <origin xyz="0 0.18 1.16" rpy="1.5708 0 0"/>
+    <origin xyz="0 0.18 1.16" rpy="-1.5708 3.14 0"/>
   </joint>
   <link name="left_J1">
@@ -121,5 +121,5 @@
     <parent link="world"/>
     <child link="right_base_link"/>
-    <origin xyz="0 -0.18 1.16" rpy="1.5708 0 3.1416"/>
+    <origin xyz="0 -0.18 1.16" rpy="1.5708 3.14 0"/>
   </joint>
   <link name="right_J1">
